File: GPU Board v1.0/Kicad/GPU Board v1.0.sch (KiCad schematic (older format))
At the start: 44 parts

Commit message: Resurrected custom part libs from .bak files and relinked them in the schematic.
Parts:
- removed U?: STM32F446ZE, symbol STM32F446ZE-RESCUE-GPU_Board_v1.0
- removed U?: IS42S16400J, symbol IS42S16400J-RESCUE-GPU_Board_v1.0
- added U?: STM32F446ZE, symbol STM32F446ZE
- added U?: IS42S16400J, symbol IS42S16400J
Changed lines of the file:
@@
 EESchema Schematic File Version 2
-LIBS:GPU Board v1.0-rescue
 LIBS:power
 LIBS:device
@@
 LIBS:IS42S16400J
 LIBS:ft813
-LIBS:GPU Board v1.0-cache
 EELAYER 25 0
 EELAYER END
@@
 Comment4 ""
 $EndDescr
-$Comp
-L STM32F446ZE-RESCUE-GPU_Board_v1.0 U?
-U 1 1 589C0060
-P 6700 5600
-F 0 "U?" H 6700 5750 60  0000 C CNN
-F 1 "STM32F446ZE" H 6700 5600 60  0000 C CNN
-F 2 "" H 5400 8600 60  0000 C CNN
-F 3 "" H 5400 8600 60  0000 C CNN
-	1    6700 5600
-	1    0    0    -1
-$EndComp
-$Comp
-L IS42S16400J-RESCUE-GPU_Board_v1.0 U?
-U 1 1 589C2926
-P 2700 3150
-F 0 "U?" H 2500 4800 60  0000 C CNN
-F 1 "IS42S16400J" H 2700 1600 60  0000 C CNN
-F 2 "" H 3200 4300 60  0000 C CNN
-F 3 "" H 3200 4300 60  0000 C CNN
-	1    2700 3150
-	1    0    0    -1
-$EndComp
 Text Label 7800 2300 0    60   ~ 0
 SD_D2
@@
 Wire Wire Line
 	9950 1700 10000 1700
+$Comp
+L STM32F446ZE U?
+U 1 1 5A5B6C21
+P 6700 5600
+F 0 "U?" H 6700 5750 60  0000 C CNN
+F 1 "STM32F446ZE" H 6700 5600 60  0000 C CNN
+F 2 "" H 5400 8600 60  0000 C CNN
+F 3 "" H 5400 8600 60  0000 C CNN
+	1    6700 5600
+	1    0    0    -1
+$EndComp
+$Comp
+L IS42S16400J U?
+U 1 1 5A5B702D
+P 2700 3150
+F 0 "U?" H 2500 4800 60  0000 C CNN
+F 1 "IS42S16400J" H 2700 1600 60  0000 C CNN
+F 2 "" H 3200 4300 60  0000 C CNN
+F 3 "" H 3200 4300 60  0000 C CNN
+	1    2700 3150
+	1    0    0    -1
+$EndComp
 $EndSCHEMATC

Commit message: update (images)
Parts:
- C? (x8): symbol CP_Small -> Device:CP_Small
- C? (x29): symbol C_Small -> Device:C_Small
- R? (x2): symbol R -> Device:R
- U?: symbol FT813 -> ft813:FT813
- U?: symbol STM32F446ZE -> stm32f446ze:STM32F446ZE
- U?: symbol IS42S16400J -> IS42S16400J:IS42S16400J
- Y? (x2): symbol Crystal_Small -> Device:Crystal_Small
Other:
- moved on the sheet: U?
