File: ZaltToISA/Kicad/ZaltToISA.sch (KiCad schematic (older format))
At the start: 10 parts

Commit message: update (images)
Parts:
- C? (x3): symbol C -> Device:C
- HDR?: symbol BUSHDR-A -> syshdr:BUSHDR-A
- HDR?: symbol BUSHDR-B -> syshdr:BUSHDR-B
- J?: symbol Bus_ISA_16bit -> ZaltToISA-rescue:Bus_ISA_16bit
- M?: symbol CY8CKIT-059 -> CY8CKIT-059:CY8CKIT-059
- U? (x3): symbol 74HC646 -> My-74-Logic:74HC646
