File: TTL VGA v0.1/Kicad/BusDecoder.sch (KiCad schematic (older format))
At the start: 11 parts, among them U16 74LS32, U17 74LS10, U18 74LS32, U8 74LS139

Commit message: TTL VGA v0.2
Parts:
- gave numbers to parts that had none: 1
Connections:
- net labels added: BusEnable
- net labels removed: ~AddressEnable
Changed lines of the file:
@@
 $Descr A4 11693 8268
 encoding utf-8
-Sheet 4 5
+Sheet 9 10
 Title "Zalt TTL VGA"
 Date "2020-02-09"
@@
 U 2 1 5E5EF2AC
 P 4150 2450
-F 0 "U8" H 4150 2817 50  0000 C CNN
+AR Path="/5E4A1CB2/5E5EE6C3/5E5EF2AC" Ref="U8"  Part="2"
+AR Path="/5ED39654/5ED6451C/5E5EF2AC" Ref="U?"  Part="2"
+F 0 "U?" H 4150 2817 50  0000 C CNN
 F 1 "74LS139" H 4150 2726 50  0000 C CNN
 F 2 "" H 4150 2450 50  0001 C CNN
@@
 ~BusDriverEnable
 Text HLabel 7250 850  0    50   Input ~ 0
-~AddressEnable
+BusEnable
 Text Notes 850  5550 0    50   ~ 0
 Z80 Bus Interface\n\n~MEMREQ~ & ~WR~ & MA19..MA12 & !~AddressEnable~\n    => Write to VRAM\n~IOREQ~ & ~WR~ & MA7..MA0 \n    => Write to Control Register\n\nControl Register:\n    A17..A12 (6 bits)\n    Options (2 bits)\n
@@
 U 1 1 5E729378
 P 6150 4150
-F 0 "U17" H 6150 4475 50  0000 C CNN
+AR Path="/5E4A1CB2/5E5EE6C3/5E729378" Ref="U17"  Part="1"
+AR Path="/5ED39654/5ED6451C/5E729378" Ref="U?"  Part="1"
+F 0 "U?" H 6150 4475 50  0000 C CNN
 F 1 "74LS10" H 6150 4384 50  0000 C CNN
 F 2 "" H 6150 4150 50  0001 C CNN
@@
 U 2 1 5E7295F8
 P 6150 2950
-F 0 "U17" H 6150 3275 50  0000 C CNN
+AR Path="/5E4A1CB2/5E5EE6C3/5E7295F8" Ref="U17"  Part="2"
+AR Path="/5ED39654/5ED6451C/5E7295F8" Ref="U?"  Part="2"
+F 0 "U?" H 6150 3275 50  0000 C CNN
 F 1 "74LS10" H 6150 3184 50  0000 C CNN
 F 2 "" H 6150 2950 50  0001 C CNN
@@
 U 3 1 5E72A784
 P 6150 3550
-F 0 "U17" H 6150 3875 50  0000 C CNN
+AR Path="/5E4A1CB2/5E5EE6C3/5E72A784" Ref="U17"  Part="3"
+AR Path="/5ED39654/5ED6451C/5E72A784" Ref="U?"  Part="3"
+F 0 "U?" H 6150 3875 50  0000 C CNN
 F 1 "74LS10" H 6150 3784 50  0000 C CNN
 F 2 "" H 6150 3550 50  0001 C CNN
@@
 U 4 1 5E72B9D2
 P 1750 6650
-F 0 "U17" H 1980 6696 50  0000 L CNN
+AR Path="/5E4A1CB2/5E5EE6C3/5E72B9D2" Ref="U17"  Part="4"
+AR Path="/5ED39654/5ED6451C/5E72B9D2" Ref="U?"  Part="4"
+F 0 "U?" H 1980 6696 50  0000 L CNN
 F 1 "74LS10" H 1980 6605 50  0000 L CNN
 F 2 "" H 1750 6650 50  0001 C CNN
@@
 U 1 1 5E72DE74
 P 7600 2600
-F 0 "U16" H 7600 2925 50  0000 C CNN
+AR Path="/5E4A1CB2/5E5EE6C3/5E72DE74" Ref="U16"  Part="1"
+AR Path="/5ED39654/5ED6451C/5E72DE74" Ref="U?"  Part="1"
+F 0 "U?" H 7600 2925 50  0000 C CNN
 F 1 "74LS32" H 7600 2834 50  0000 C CNN
 F 2 "" H 7600 2600 50  0001 C CNN
@@
 U 2 1 5E72E692
 P 6150 2250
-F 0 "U16" H 6150 2575 50  0000 C CNN
+AR Path="/5E4A1CB2/5E5EE6C3/5E72E692" Ref="U16"  Part="2"
+AR Path="/5ED39654/5ED6451C/5E72E692" Ref="U?"  Part="2"
+F 0 "U?" H 6150 2575 50  0000 C CNN
 F 1 "74LS32" H 6150 2484 50  0000 C CNN
 F 2 "" H 6150 2250 50  0001 C CNN
@@
 U 3 1 5E72F764
 P 6900 3250
-F 0 "U16" H 6900 3575 50  0000 C CNN
+AR Path="/5E4A1CB2/5E5EE6C3/5E72F764" Ref="U16"  Part="3"
+AR Path="/5ED39654/5ED6451C/5E72F764" Ref="U?"  Part="3"
+F 0 "U?" H 6900 3575 50  0000 C CNN
 F 1 "74LS32" H 6900 3484 50  0000 C CNN
 F 2 "" H 6900 3250 50  0001 C CNN
@@
 U 4 1 5E730954
 P 7800 4550
-F 0 "U16" H 7800 4875 50  0000 C CNN
+AR Path="/5E4A1CB2/5E5EE6C3/5E730954" Ref="U16"  Part="4"
+AR Path="/5ED39654/5ED6451C/5E730954" Ref="U?"  Part="4"
+F 0 "U?" H 7800 4875 50  0000 C CNN
 F 1 "74LS32" H 7800 4784 50  0000 C CNN
 F 2 "" H 7800 4550 50  0001 C CNN
@@
 U 5 1 5E7317BD
 P 2600 6650
-F 0 "U16" H 2830 6696 50  0000 L CNN
+AR Path="/5E4A1CB2/5E5EE6C3/5E7317BD" Ref="U16"  Part="5"
+AR Path="/5ED39654/5ED6451C/5E7317BD" Ref="U?"  Part="5"
+F 0 "U?" H 2830 6696 50  0000 L CNN
 F 1 "74LS32" H 2830 6605 50  0000 L CNN
 F 2 "" H 2600 6650 50  0001 C CNN
@@
 U 1 1 5E74F207
 P 5400 4700
-F 0 "U18" H 5400 5025 50  0000 C CNN
+AR Path="/5E4A1CB2/5E5EE6C3/5E74F207" Ref="U18"  Part="1"
+AR Path="/5ED39654/5ED6451C/5E74F207" Ref="U?"  Part="1"
+F 0 "U?" H 5400 5025 50  0000 C CNN
 F 1 "74LS32" H 5400 4934 50  0000 C CNN
 F 2 "" H 5400 4700 50  0001 C CNN
@@
 U 2 1 5E751B18
 P 5400 5250
-F 0 "U18" H 5400 5575 50  0000 C CNN
+AR Path="/5E4A1CB2/5E5EE6C3/5E751B18" Ref="U18"  Part="2"
+AR Path="/5ED39654/5ED6451C/5E751B18" Ref="U?"  Part="2"
+F 0 "U?" H 5400 5575 50  0000 C CNN
 F 1 "74LS32" H 5400 5484 50  0000 C CNN
 F 2 "" H 5400 5250 50  0001 C CNN
@@
 U 4 1 5E753738
 P 6150 5000
-F 0 "U18" H 6150 5325 50  0000 C CNN
+AR Path="/5E4A1CB2/5E5EE6C3/5E753738" Ref="U18"  Part="4"
+AR Path="/5ED39654/5ED6451C/5E753738" Ref="U?"  Part="4"
+F 0 "U?" H 6150 5325 50  0000 C CNN
 F 1 "74LS32" H 6150 5234 50  0000 C CNN
 F 2 "" H 6150 5000 50  0001 C CNN
@@
 U 3 1 5E7560E1
 P 6950 4450
-F 0 "U18" H 6950 4775 50  0000 C CNN
+AR Path="/5E4A1CB2/5E5EE6C3/5E7560E1" Ref="U18"  Part="3"
+AR Path="/5ED39654/5ED6451C/5E7560E1" Ref="U?"  Part="3"
+F 0 "U?" H 6950 4775 50  0000 C CNN
 F 1 "74LS32" H 6950 4684 50  0000 C CNN
 F 2 "" H 6950 4450 50  0001 C CNN
@@
 U 5 1 5E75841D
 P 3400 6650
-F 0 "U18" H 3630 6696 50  0000 L CNN
+AR Path="/5E4A1CB2/5E5EE6C3/5E75841D" Ref="U18"  Part="5"
+AR Path="/5ED39654/5ED6451C/5E75841D" Ref="U?"  Part="5"
+F 0 "U?" H 3630 6696 50  0000 L CNN
 F 1 "74LS32" H 3630 6605 50  0000 L CNN
 F 2 "" H 3400 6650 50  0001 C CNN
@@
 U 1 1 5E7AF347
 P 3000 5950
-F 0 "#PWR035" H 3000 5800 50  0001 C CNN
+AR Path="/5E4A1CB2/5E5EE6C3/5E7AF347" Ref="#PWR035"  Part="1"
+AR Path="/5ED39654/5ED6451C/5E7AF347" Ref="#PWR?"  Part="1"
+F 0 "#PWR?" H 3000 5800 50  0001 C CNN
 F 1 "+5V" H 3015 6123 50  0000 C CNN
 F 2 "" H 3000 5950 50  0001 C CNN
@@
 U 1 1 5E7B0259
 P 3000 7300
-F 0 "#PWR036" H 3000 7050 50  0001 C CNN
+AR Path="/5E4A1CB2/5E5EE6C3/5E7B0259" Ref="#PWR036"  Part="1"
+AR Path="/5ED39654/5ED6451C/5E7B0259" Ref="#PWR?"  Part="1"
+F 0 "#PWR?" H 3000 7050 50  0001 C CNN
 F 1 "GND" H 3005 7127 50  0000 C CNN
 F 2 "" H 3000 7300 50  0001 C CNN
@@
 U 1 1 5E7B85F7
 P 1400 6200
-F 0 "C9" H 1515 6246 50  0000 L CNN
+AR Path="/5E4A1CB2/5E5EE6C3/5E7B85F7" Ref="C9"  Part="1"
+AR Path="/5ED39654/5ED6451C/5E7B85F7" Ref="C?"  Part="1"
+F 0 "C?" H 1515 6246 50  0000 L CNN
 F 1 "C" H 1515 6155 50  0000 L CNN
 F 2 "" H 1438 6050 50  0001 C CNN
@@
 U 1 1 5E7B914A
 P 2200 6200
-F 0 "C10" H 2315 6246 50  0000 L CNN
+AR Path="/5E4A1CB2/5E5EE6C3/5E7B914A" Ref="C10"  Part="1"
+AR Path="/5ED39654/5ED6451C/5E7B914A" Ref="C?"  Part="1"
+F 0 "C?" H 2315 6246 50  0000 L CNN
 F 1 "C" H 2315 6155 50  0000 L CNN
 F 2 "" H 2238 6050 50  0001 C CNN
@@
 U 1 1 5E7B947A
 P 3000 6200
-F 0 "C11" H 3115 6246 50  0000 L CNN
+AR Path="/5E4A1CB2/5E5EE6C3/5E7B947A" Ref="C11"  Part="1"
+AR Path="/5ED39654/5ED6451C/5E7B947A" Ref="C?"  Part="1"
+F 0 "C?" H 3115 6246 50  0000 L CNN
 F 1 "C" H 3115 6155 50  0000 L CNN
 F 2 "" H 3038 6050 50  0001 C CNN
@@
 MA2
 $Comp
-L 74xx:74LS00 U?
+L 74xx:74LS00 U15
 U 1 1 5E61D130
 P 8750 1200
+AR Path="/5E4A1CB2/5E5EE6C3/5E61D130" Ref="U15"  Part="1"
+AR Path="/5ED39654/5ED6451C/5E61D130" Ref="U?"  Part="1"
 F 0 "U?" H 8750 1525 50  0000 C CNN
 F 1 "74LS00" H 8750 1434 50  0000 C CNN
@@
 $EndComp
 $Comp
-L 74xx:74LS00 U?
+L 74xx:74LS00 U15
 U 2 1 5E628EB2
 P 9450 1750
+AR Path="/5E4A1CB2/5E5EE6C3/5E628EB2" Ref="U15"  Part="2"
+AR Path="/5ED39654/5ED6451C/5E628EB2" Ref="U?"  Part="2"
 F 0 "U?" H 9450 2075 50  0000 C CNN
 F 1 "74LS00" H 9450 1984 50  0000 C CNN
@@
 $EndComp
 $Comp
-L 74xx:74LS00 U?
+L 74xx:74LS00 U15
 U 3 1 5E62BDF3
 P 8600 2500
+AR Path="/5E4A1CB2/5E5EE6C3/5E62BDF3" Ref="U15"  Part="3"
+AR Path="/5ED39654/5ED6451C/5E62BDF3" Ref="U?"  Part="3"
 F 0 "U?" H 8600 2825 50  0000 C CNN
 F 1 "74LS00" H 8600 2734 50  0000 C CNN
@@
 $EndComp
 $Comp
-L 74xx:74LS00 U?
+L 74xx:74LS00 U15
 U 4 1 5E62EF03
 P 8650 4550
+AR Path="/5E4A1CB2/5E5EE6C3/5E62EF03" Ref="U15"  Part="4"
+AR Path="/5ED39654/5ED6451C/5E62EF03" Ref="U?"  Part="4"
 F 0 "U?" H 8650 4875 50  0000 C CNN
 F 1 "74LS00" H 8650 4784 50  0000 C CNN
