File: TTL VGA v0.2/Kicad/NewBusDecoder.sch (KiCad schematic (older format))
At the start: 0 parts

Commit message: update kicad
Other:
- note added: "CPU access to the Video Memort Bus"
- note added: "CPU interface"
- note added: "Low and High address of the scroll register strobe.\nValue loaded when the line counters reset."
- note added: "Pallette Register for selecting an active color pallete."
- note added: "Signals that control VGA behavior\n-Video Mode"
- note added: "TODO: CPU access to the content of the Pallete"
- note added: "VGA video is active"
- note added: "VRAM bank register strobe"
Changed lines of the file:
@@
 Text HLabel 6650 5250 2    50   Output ~ 0
 Settings
+Text HLabel 9500 4000 2    50   Output ~ 0
+~PalleteRegStrobe
+Text Notes 9100 1600 0    50   ~ 0
+VRAM bank register strobe
+Text Notes 8050 3450 0    50   ~ 0
+CPU access to the Video Memort Bus
+Text Notes 8050 3750 0    50   ~ 0
+TODO: CPU access to the content of the Pallete
+Text Notes 7350 4000 0    50   ~ 0
+Pallette Register for selecting an active color pallete.
+Text Notes 7350 4500 0    50   ~ 0
+Low and High address of the scroll register strobe.\nValue loaded when the line counters reset.
+Text Notes 6200 5500 0    50   ~ 0
+Signals that control VGA behavior\n-Video Mode
+Text Notes 9000 2850 0    50   ~ 0
+VGA video is active
+Text Notes 1500 2450 0    50   ~ 0
+CPU interface
 $EndSCHEMATC

Commit message: Update
Other:
- note added: "TODO"
- note added: "This module decodes IO addresses for the Z80 CPU to access various parts of the VGA adapter.\n\n- VRAM banks (4k)\n- Video Modes\n- Color Palette"
Changed lines of the file:
@@
 Text Notes 1500 2450 0    50   ~ 0
 CPU interface
+Text Notes 850  1100 0    50   ~ 0
+This module decodes IO addresses for the Z80 CPU to access various parts of the VGA adapter.\n\n- VRAM banks (4k)\n- Video Modes\n- Color Palette
+Text Notes 3200 4000 0    866  ~ 173
+TODO
 $EndSCHEMATC
