File: TTL VGA v0.2/Kicad/VideoMemory.sch (KiCad schematic (older format))
At the start: 3 parts

Commit message: Update
Other:
- note added: "Active when the CPU has write-access"
- note added: "Active when the VGA adapter \nis output VRAM data to the screen."
- note added: "This module contains the VRAM.\n2x 64kB at this time."
Changed lines of the file:
@@
 Wire Bus Line
 	2700 1350 2700 6100
+Text Notes 7100 1100 0    49   ~ 0
+This module contains the VRAM.\n2x 64kB at this time.
+Text Notes 1250 5250 0    49   ~ 0
+Active when the VGA adapter \nis output VRAM data to the screen.
+Text Notes 1050 5900 0    49   ~ 0
+Active when the CPU has write-access
 $EndSCHEMATC
