File: TTL VGA v0.2/Kicad/VideoModes.sch (KiCad schematic (older format))
At the start: 7 parts

Commit message: update kicad
Connections:
- net labels removed: MA17, MA18
- wire segments 153 -> 151
Other:
- note added: "Based on Opt0/1 one of 4 Video Modes is selected.\nEverything is based of the 640x480@60Hz timing.\nThe VRAM Address Counter counts visible pixels.\nEach Video Mode maps these pixel addresses to VRAM addresses.\nVM0:off\nVM1: 256x192 - 2 colors (1 bit per pixel)\nVM2: 256x192 - 4 colors (2 bits per pixel)\nVM3: 256x192 - 16 colors (4 bits per pixel)\n"
- note removed: "Based on Opt0/1 one of 4 Video Modes is selected.\nEverything is based of the 640x480@60Hz timing.\nThe VRAM Address Counter counts visible pixels.\nEach Video Mode maps these pixel addresses to VRAM addresses.\nVM0:off\nVM1: 256x192 - 16 colors (4 bits per pixel)\nVM2: 256x192 - 4 colors (2 bits per pixel)\nVM3: 256x192 - 2 colors (1 bit per pixel)\n"
Changed lines of the file:
@@
 Entry Wire Line
 	9350 3200 9450 3100
-Entry Wire Line
-	9350 3300 9450 3200
-Entry Wire Line
-	9350 3400 9450 3300
 Wire Wire Line
 	9450 1500 10050 1500
@@
 Wire Wire Line
 	9450 3100 10050 3100
-Wire Wire Line
-	9450 3200 10050 3200
-Wire Wire Line
-	9450 3300 10050 3300
 Text Label 9750 1500 0    50   ~ 0
 MA0
@@
 Text Label 9750 3100 0    50   ~ 0
 MA16
-Text Label 9750 3200 0    50   ~ 0
-MA17
-Text Label 9750 3300 0    50   ~ 0
-MA18
 Text Notes 9700 1250 0    50   ~ 0
 To VRAM
@@
 A11
 Text Notes 4000 7350 0    50   ~ 0
-Based on Opt0/1 one of 4 Video Modes is selected.\nEverything is based of the 640x480@60Hz timing.\nThe VRAM Address Counter counts visible pixels.\nEach Video Mode maps these pixel addresses to VRAM addresses.\nVM0:off\nVM1: 256x192 - 16 colors (4 bits per pixel)\nVM2: 256x192 - 4 colors (2 bits per pixel)\nVM3: 256x192 - 2 colors (1 bit per pixel)\n
+Based on Opt0/1 one of 4 Video Modes is selected.\nEverything is based of the 640x480@60Hz timing.\nThe VRAM Address Counter counts visible pixels.\nEach Video Mode maps these pixel addresses to VRAM addresses.\nVM0:off\nVM1: 256x192 - 2 colors (1 bit per pixel)\nVM2: 256x192 - 4 colors (2 bits per pixel)\nVM3: 256x192 - 16 colors (4 bits per pixel)\n
 Text HLabel 1200 4300 0    50   Input ~ 0
 PixelAddress

Commit message: Update
Other:
- note added: "Mode 0: \ndisengage driving the \nVRAM / CPU access\n(reserved for text mode)\n\nMode 1: \nA0 selects pixel data\nA8 duplicate line\n\nA1-A7 => A0-A6\nA9-A18 => A7-A16\n\nMode 2:\nA0,A1 selects pixel data\nA9 duplicate line\n\nA2-A8 => A0-A6\nA10-A18 => A7-A15\n\nMode 3:\nA0,A1,A2 selects pixel data\nA10 duplicate line\n\nA3-A9 => A0-A6\nA11-A18 => A7-A14\n"
- note added: "This module implements the VRAM address control for the different Video Modes.\nThe incoming Pixel-Address is mapped to an actual VRAM address.\nEach video mode uses a different combination of Pixel-Address lines, \nbecause each Video Mode uses a different number of bits per pixel.\nAlso, the same horizontal line is duplicated. That means that the VRAM \naddresses for each (pixel) line on the scr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"
- note added: "Video Mode 1"
- note added: "Video Mode 2"
- note added: "Video Mode 3"
- note removed: "Mode 0: \ndisengage driving the \nVRAM / CPU access\n\nMode 1: \nA0 selects pixel data\nA8 duplicate line\n\nA1-A7 => A0-A6\nA9-A18 => A7-A16\n\nMode 2:\nA0,A1 selects pixel data\nA9 duplicate line\n\nA2-A8 => A0-A6\nA10-A18 => A7-A15\n\nMode 3:\nA0,A1,A2 selects pixel data\nA10 duplicate line\n\nA3-A9 => A0-A6\nA11-A18 => A7-A14\n"
Changed lines of the file:
@@
 From VRAM\nAddress Counter
 Text Notes 10000 6300 0    50   ~ 0
-Mode 0: \ndisengage driving the \nVRAM / CPU access\n\nMode 1: \nA0 selects pixel data\nA8 duplicate line\n\nA1-A7 => A0-A6\nA9-A18 => A7-A16\n\nMode 2:\nA0,A1 selects pixel data\nA9 duplicate line\n\nA2-A8 => A0-A6\nA10-A18 => A7-A15\n\nMode 3:\nA0,A1,A2 selects pixel data\nA10 duplicate line\n\nA3-A9 => A0-A6\nA11-A18 => A7-A14\n
+Mode 0: \ndisengage driving the \nVRAM / CPU access\n(reserved for text mode)\n\nMode 1: \nA0 selects pixel data\nA8 duplicate line\n\nA1-A7 => A0-A6\nA9-A18 => A7-A16\n\nMode 2:\nA0,A1 selects pixel data\nA9 duplicate line\n\nA2-A8 => A0-A6\nA10-A18 => A7-A15\n\nMode 3:\nA0,A1,A2 selects pixel data\nA10 duplicate line\n\nA3-A9 => A0-A6\nA11-A18 => A7-A14\n
 $Comp
 L 74xx:74LS245 U?
@@
 Wire Bus Line
 	9350 1600 9350 4050
+Text Notes 5950 6150 0    49   ~ 0
+This module implements the VRAM address control for the different Video Modes.\nThe incoming Pixel-Address is mapped to an actual VRAM address.\nEach video mode uses a different combination of Pixel-Address lines, \nbecause each Video Mode uses a different number of bits per pixel.\nAlso, the same horizontal line is duplicated. That means that the VRAM \naddresses for each (pixel) line on the screen are accessed twice.\nThis is done by simply ignoring a single Pixel-Address line (A8/A9/A10)
+Text Notes 2950 1000 0    49   ~ 0
+Video Mode 1
+Text Notes 5000 1000 0    49   ~ 0
+Video Mode 2
+Text Notes 7300 1000 0    49   ~ 0
+Video Mode 3
 $EndSCHEMATC
