File: Under Construction/VDP-Composite v0.1/Kicad/VRAM.sch (KiCad schematic (older format))
At the start: 12 parts, among them U301 D41464, U302 D41464, U303 D41464, U304 D41464, U305 D41464, U306 D41464

Commit message: progress
Parts:
- C301, C302, C303, C304, C305, C306: footprint Capacitor_SMD:C_1206_3216Metric_Pad1.33x1.80mm_HandSolder -> Capacitor_SMD:C_0603_1608Metric_Pad1.08x0.95mm_HandSolder
Changed lines of the file:
@@
 $Descr A4 11693 8268
 encoding utf-8
-Sheet 3 3
+Sheet 3 4
 Title ""
 Date ""
@@
 F 0 "C301" H 2215 6696 50  0000 L CNN
 F 1 "100nF" H 2215 6605 50  0000 L CNN
-F 2 "Capacitor_SMD:C_1206_3216Metric_Pad1.33x1.80mm_HandSolder" H 2138 6500 50  0001 C CNN
+F 2 "Capacitor_SMD:C_0603_1608Metric_Pad1.08x0.95mm_HandSolder" H 2138 6500 50  0001 C CNN
 F 3 "~" H 2100 6650 50  0001 C CNN
 	1    2100 6650
@@
 F 0 "C302" H 2815 6696 50  0000 L CNN
 F 1 "100nF" H 2815 6605 50  0000 L CNN
-F 2 "Capacitor_SMD:C_1206_3216Metric_Pad1.33x1.80mm_HandSolder" H 2738 6500 50  0001 C CNN
+F 2 "Capacitor_SMD:C_0603_1608Metric_Pad1.08x0.95mm_HandSolder" H 2738 6500 50  0001 C CNN
 F 3 "~" H 2700 6650 50  0001 C CNN
 	1    2700 6650
@@
 F 0 "C303" H 3365 6696 50  0000 L CNN
 F 1 "100nF" H 3365 6605 50  0000 L CNN
-F 2 "Capacitor_SMD:C_1206_3216Metric_Pad1.33x1.80mm_HandSolder" H 3288 6500 50  0001 C CNN
+F 2 "Capacitor_SMD:C_0603_1608Metric_Pad1.08x0.95mm_HandSolder" H 3288 6500 50  0001 C CNN
 F 3 "~" H 3250 6650 50  0001 C CNN
 	1    3250 6650
@@
 F 0 "C304" H 3915 6696 50  0000 L CNN
 F 1 "100nF" H 3915 6605 50  0000 L CNN
-F 2 "Capacitor_SMD:C_1206_3216Metric_Pad1.33x1.80mm_HandSolder" H 3838 6500 50  0001 C CNN
+F 2 "Capacitor_SMD:C_0603_1608Metric_Pad1.08x0.95mm_HandSolder" H 3838 6500 50  0001 C CNN
 F 3 "~" H 3800 6650 50  0001 C CNN
 	1    3800 6650
@@
 F 0 "C305" H 4465 6696 50  0000 L CNN
 F 1 "100nF" H 4465 6605 50  0000 L CNN
-F 2 "Capacitor_SMD:C_1206_3216Metric_Pad1.33x1.80mm_HandSolder" H 4388 6500 50  0001 C CNN
+F 2 "Capacitor_SMD:C_0603_1608Metric_Pad1.08x0.95mm_HandSolder" H 4388 6500 50  0001 C CNN
 F 3 "~" H 4350 6650 50  0001 C CNN
 	1    4350 6650
@@
 F 0 "C306" H 5015 6696 50  0000 L CNN
 F 1 "100nF" H 5015 6605 50  0000 L CNN
-F 2 "Capacitor_SMD:C_1206_3216Metric_Pad1.33x1.80mm_HandSolder" H 4938 6500 50  0001 C CNN
+F 2 "Capacitor_SMD:C_0603_1608Metric_Pad1.08x0.95mm_HandSolder" H 4938 6500 50  0001 C CNN
 F 3 "~" H 4900 6650 50  0001 C CNN
 	1    4900 6650
