File: Under Construction/VDP-Composite v0.1/Kicad/SoundGen.sch (KiCad schematic (older format))
At the start: 19 parts, among them J401 Ports, U202 74HCT04, U401 YM2149, Y401 2-4MHz

Commit message: updates
Parts:
- C402, C403: value 470uF -> 220uF; footprint Capacitor_SMD:CP_Elec_5x3 -> Capacitor_SMD:CP_Elec_6.3x7.7
Changed lines of the file:
@@
 P 9100 1650
 F 0 "C402" V 9325 1650 50  0000 C CNN
-F 1 "470uF" V 9234 1650 50  0000 C CNN
-F 2 "Capacitor_SMD:CP_Elec_5x3" H 9100 1650 50  0001 C CNN
+F 1 "220uF" V 9234 1650 50  0000 C CNN
+F 2 "Capacitor_SMD:CP_Elec_6.3x7.7" H 9100 1650 50  0001 C CNN
 F 3 "~" H 9100 1650 50  0001 C CNN
 	1    9100 1650
@@
 P 9100 2000
 F 0 "C403" V 9325 2000 50  0000 C CNN
-F 1 "470uF" V 9234 2000 50  0000 C CNN
-F 2 "Capacitor_SMD:CP_Elec_5x3" H 9100 2000 50  0001 C CNN
+F 1 "220uF" V 9234 2000 50  0000 C CNN
+F 2 "Capacitor_SMD:CP_Elec_6.3x7.7" H 9100 2000 50  0001 C CNN
 F 3 "~" H 9100 2000 50  0001 C CNN
 	1    9100 2000
