File: Under Construction/VDP-Composite v0.1/Kicad/VDP-Composite.kicad_pcb (KiCad board)
At the start: 2 copper layers, 99.7 x 99.7 mm, 19 parts, among them J101 Screw_Terminal_01x02, U101 G22V10, U102 74HCT574, U201 v9958, U202 74HCT04, U203 CXA1645, U301 D41464, U302 D41464, U303 D41464, U304 D41464, U305 D41464, U306 D41464, Y201 21.47727MHz

Commit message: progress
Parts:
- added C101: 100nF, Capacitor_SMD:C_0603_1608Metric_Pad1.08x0.95mm_HandSolder, B.Cu at (74.3, 150.2)
- added C102: 100nF, Capacitor_SMD:C_0603_1608Metric_Pad1.08x0.95mm_HandSolder, B.Cu at (100.5, 173.4)
- added C201: 30pF, Capacitor_THT:C_Disc_D6.0mm_W4.4mm_P5.00mm, F.Cu at (107.4, 146.1)
- added C202: 22pF, Capacitor_SMD:C_0603_1608Metric_Pad1.08x0.95mm_HandSolder, B.Cu at (117.3, 145.0)
- added C203: 22pF, Capacitor_SMD:C_0603_1608Metric_Pad1.08x0.95mm_HandSolder, F.Cu at (124.5, 215.9)
- added C204: 30pF, Capacitor_THT:C_Disc_D6.0mm_W4.4mm_P5.00mm, F.Cu at (139.2, 215.9)
- added C205: 100nF, Capacitor_SMD:C_0603_1608Metric_Pad1.08x0.95mm_HandSolder, B.Cu at (117.0, 208.3)
- added C206: 100nF, Capacitor_SMD:C_0603_1608Metric_Pad1.08x0.95mm_HandSolder, B.Cu at (87.1, 210.1)
- added C207: *27/18pF, Capacitor_SMD:C_0603_1608Metric_Pad1.08x0.95mm_HandSolder, B.Cu at (89.7, 220.2)
- added C208: 100nF, Capacitor_SMD:C_0603_1608Metric_Pad1.08x0.95mm_HandSolder, B.Cu at (102.9, 194.0)
- added C209: 10uF, Capacitor_SMD:CP_Elec_4x3, F.Cu at (82.8, 209.1)
- added C210: 100nF, Capacitor_SMD:C_0603_1608Metric_Pad1.08x0.95mm_HandSolder, B.Cu at (102.9, 187.2)
- added C211: 100nF, Capacitor_SMD:C_0603_1608Metric_Pad1.08x0.95mm_HandSolder, B.Cu at (102.9, 190.6)
- added C212: 100nF, Capacitor_SMD:C_0603_1608Metric_Pad1.08x0.95mm_HandSolder, B.Cu at (104.9, 210.1)
- added C213: 100nF, Capacitor_SMD:C_0603_1608Metric_Pad1.08x0.95mm_HandSolder, B.Cu at (105.3, 216.2)
- added C214: 100nF, Capacitor_SMD:C_0603_1608Metric_Pad1.08x0.95mm_HandSolder, B.Cu at (99.8, 210.1)
- added C215: 4.7pF, Capacitor_SMD:C_0603_1608Metric_Pad1.08x0.95mm_HandSolder, B.Cu at (94.7, 216.9)
- added C216: 47pF, Capacitor_SMD:C_0603_1608Metric_Pad1.08x0.95mm_HandSolder, B.Cu at (84.6, 210.1)
- added C217: 220uF, Capacitor_SMD:CP_Elec_4x3, F.Cu at (64.8, 200.7)
- added C218: 220uF, Capacitor_SMD:CP_Elec_4x3, F.Cu at (64.8, 226.1)
- added C219: 220uF, Capacitor_SMD:CP_Elec_4x3, F.Cu at (64.8, 205.8)
- added C220: 220uF, Capacitor_SMD:CP_Elec_4x3, F.Cu at (64.8, 221.0)
- added C221: 220uF, Capacitor_SMD:CP_Elec_4x3, F.Cu at (64.8, 210.8)
- added C222: 220uF, Capacitor_SMD:CP_Elec_4x3, F.Cu at (64.8, 215.9)
- added C223: 100nF, Capacitor_SMD:C_0603_1608Metric_Pad1.08x0.95mm_HandSolder, B.Cu at (113.8, 160.6)
- added C224: 100nF, Capacitor_SMD:C_0603_1608Metric_Pad1.08x0.95mm_HandSolder, B.Cu at (94.7, 185.9)
- added C225: 100nF, Capacitor_SMD:C_0603_1608Metric_Pad1.08x0.95mm_HandSolder, B.Cu at (124.5, 231.4)
- added C226: 100nF, Capacitor_SMD:C_0603_1608Metric_Pad1.08x0.95mm_HandSolder, B.Cu at (79.5, 209.8)
- added C227: 100nF, Capacitor_SMD:C_0603_1608Metric_Pad1.08x0.95mm_HandSolder, B.Cu at (94.7, 220.2)
- added C301: 100nF, Capacitor_SMD:C_0603_1608Metric_Pad1.08x0.95mm_HandSolder, B.Cu at (121.3, 149.0)
- added C302: 100nF, Capacitor_SMD:C_0603_1608Metric_Pad1.08x0.95mm_HandSolder, B.Cu at (121.0, 160.4)
- added C303: 100nF, Capacitor_SMD:C_0603_1608Metric_Pad1.08x0.95mm_HandSolder, B.Cu at (121.2, 171.9)
- added C304: 100nF, Capacitor_SMD:C_0603_1608Metric_Pad1.08x0.95mm_HandSolder, B.Cu at (121.0, 183.3)
- added C305: 100nF, Capacitor_SMD:C_0603_1608Metric_Pad1.08x0.95mm_HandSolder, B.Cu at (121.0, 194.7)
- added C306: 100nF, Capacitor_SMD:C_0603_1608Metric_Pad1.08x0.95mm_HandSolder, B.Cu at (121.0, 206.1)
- added C401: 100nF, Capacitor_SMD:C_0603_1608Metric_Pad1.08x0.95mm_HandSolder, B.Cu at (89.1, 151.1)
- added C402: 470uF, Capacitor_SMD:CP_Elec_5x3, F.Cu at (65.3, 195.1)
- added C403: 470uF, Capacitor_SMD:CP_Elec_5x3, F.Cu at (65.3, 189.0)
- added C404: 22pF, Capacitor_SMD:C_0603_1608Metric_Pad1.08x0.95mm_HandSolder, F.Cu at (124.5, 222.3)
- added C405: 30pF, Capacitor_THT:C_Disc_D6.0mm_W4.4mm_P5.00mm, F.Cu at (139.2, 222.3)
- added J207: AVConn, Connector_IDC:IDC-Header_2x10_P2.54mm_Horizontal, F.Cu at (59.1, 218.4)
- added J401: Ports, Connector_PinHeader_2.54mm:PinHeader_2x10_P2.54mm_Vertical, F.Cu at (52.8, 174.0)
- added JP101: Vector-Enable, Jumper:SolderJumper-3_P1.3mm_Open_RoundedPad1.0x1.5mm, B.Cu at (68.0, 180.0)
- added JP201: NTSC/PAL, Jumper:SolderJumper-3_P1.3mm_Open_RoundedPad1.0x1.5mm, B.Cu at (92.2, 210.3)
- added JP202: NTSC/PAL, Jumper:SolderJumper-3_P1.3mm_Open_RoundedPad1.0x1.5mm, B.Cu at (110.8, 209.2)
- added JP401: Clock/2, Jumper:SolderJumper-2_P1.3mm_Open_RoundedPad1.0x1.5mm, B.Cu at (89.6, 186.0)
- added R101: 10k, Resistor_SMD:R_0603_1608Metric_Pad0.98x0.95mm_HandSolder, B.Cu at (72.4, 182.1)
- added R201: 470k, Resistor_SMD:R_0603_1608Metric_Pad0.98x0.95mm_HandSolder, B.Cu at (116.4, 148.8)
- added R202: 10k, Resistor_SMD:R_0603_1608Metric_Pad0.98x0.95mm_HandSolder, B.Cu at (101.0, 152.9)
- added R203: 10k, Resistor_SMD:R_0603_1608Metric_Pad0.98x0.95mm_HandSolder, B.Cu at (101.0, 154.7)
- added R204: 10k, Resistor_SMD:R_0603_1608Metric_Pad0.98x0.95mm_HandSolder, B.Cu at (100.8, 183.2)
- added R205: 10k, Resistor_SMD:R_0603_1608Metric_Pad0.98x0.95mm_HandSolder, B.Cu at (100.8, 181.4)
- added R206: 10k, Resistor_SMD:R_0603_1608Metric_Pad0.98x0.95mm_HandSolder, B.Cu at (100.8, 179.6)
- added R207: 10k, Resistor_SMD:R_0603_1608Metric_Pad0.98x0.95mm_HandSolder, B.Cu at (100.8, 177.9)
- added R208: 10k, Resistor_SMD:R_0603_1608Metric_Pad0.98x0.95mm_HandSolder, B.Cu at (100.8, 176.0)
- added R209: 10k, Resistor_SMD:R_0603_1608Metric_Pad0.98x0.95mm_HandSolder, B.Cu at (100.3, 169.9)
- added R210: 10k, Resistor_SMD:R_0603_1608Metric_Pad0.98x0.95mm_HandSolder, B.Cu at (95.1, 171.5)
- added R211: 10k, Resistor_SMD:R_0603_1608Metric_Pad0.98x0.95mm_HandSolder, B.Cu at (100.3, 166.5)
- added R212: 10k, Resistor_SMD:R_0603_1608Metric_Pad0.98x0.95mm_HandSolder, B.Cu at (101.0, 156.5)
- added R213: 10k, Resistor_SMD:R_0603_1608Metric_Pad0.98x0.95mm_HandSolder, B.Cu at (102.0, 184.7)
- added R214: 1k, Resistor_SMD:R_0603_1608Metric_Pad0.98x0.95mm_HandSolder, B.Cu at (133.1, 218.5)
- added R215: 1M, Resistor_SMD:R_0603_1608Metric_Pad0.98x0.95mm_HandSolder, B.Cu at (129.5, 218.5)
- added R216: 10k, Resistor_SMD:R_0603_1608Metric_Pad0.98x0.95mm_HandSolder, B.Cu at (101.0, 161.8)
- added R217: 470, Resistor_SMD:R_0603_1608Metric_Pad0.98x0.95mm_HandSolder, B.Cu at (101.0, 158.2)
- added R218: 10k, Resistor_SMD:R_0603_1608Metric_Pad0.98x0.95mm_HandSolder, B.Cu at (101.0, 160.0)
- added R219: *20/16k, Resistor_SMD:R_0603_1608Metric_Pad0.98x0.95mm_HandSolder, B.Cu at (92.2, 220.2)
- added R220: 1k, Resistor_SMD:R_0603_1608Metric_Pad0.98x0.95mm_HandSolder, B.Cu at (107.4, 209.6)
- added R221: 2.2k, Resistor_SMD:R_0603_1608Metric_Pad0.98x0.95mm_HandSolder, B.Cu at (95.8, 210.1)
- added R222: 470, Resistor_SMD:R_0603_1608Metric_Pad0.98x0.95mm_HandSolder, B.Cu at (100.0, 194.1)
- added R223: 470, Resistor_SMD:R_0603_1608Metric_Pad0.98x0.95mm_HandSolder, B.Cu at (100.0, 187.3)
- added R224: 47k, Resistor_SMD:R_0603_1608Metric_Pad0.98x0.95mm_HandSolder, B.Cu at (82.0, 220.2)
- added R225: 470, Resistor_SMD:R_0603_1608Metric_Pad0.98x0.95mm_HandSolder, B.Cu at (100.0, 190.7)
- added R226: 75, Resistor_SMD:R_0603_1608Metric_Pad0.98x0.95mm_HandSolder, F.Cu at (70.4, 200.7)
- added R227: 75, Resistor_SMD:R_0603_1608Metric_Pad0.98x0.95mm_HandSolder, F.Cu at (70.4, 223.9)
- added R228: 75, Resistor_SMD:R_0603_1608Metric_Pad0.98x0.95mm_HandSolder, F.Cu at (70.4, 205.8)
- added R229: 75, Resistor_SMD:R_0603_1608Metric_Pad0.98x0.95mm_HandSolder, F.Cu at (70.3, 221.0)
- added R230: 75, Resistor_SMD:R_0603_1608Metric_Pad0.98x0.95mm_HandSolder, F.Cu at (70.4, 210.8)
- added R231: 75, Resistor_SMD:R_0603_1608Metric_Pad0.98x0.95mm_HandSolder, F.Cu at (70.4, 216.0)
- added R232: 1k, Resistor_SMD:R_0603_1608Metric_Pad0.98x0.95mm_HandSolder, B.Cu at (63.2, 204.2)
- added R233: 10k, Resistor_SMD:R_0603_1608Metric_Pad0.98x0.95mm_HandSolder, B.Cu at (61.5, 204.2)
- added R234: 120, Resistor_SMD:R_0603_1608Metric_Pad0.98x0.95mm_HandSolder, B.Cu at (63.2, 199.7)
- added R235: 180, Resistor_SMD:R_0603_1608Metric_Pad0.98x0.95mm_HandSolder, B.Cu at (61.5, 199.7)
- added R236: 1k, Resistor_SMD:R_0603_1608Metric_Pad0.98x0.95mm_HandSolder, B.Cu at (92.5, 208.1)
- added R401: 3k, Resistor_SMD:R_0603_1608Metric_Pad0.98x0.95mm_HandSolder, B.Cu at (88.8, 154.5)
- added R402: 3k, Resistor_SMD:R_0603_1608Metric_Pad0.98x0.95mm_HandSolder, B.Cu at (80.3, 159.5)
- added R403: 3k, Resistor_SMD:R_0603_1608Metric_Pad0.98x0.95mm_HandSolder, B.Cu at (80.3, 154.5)
- added R404: 1k6, Resistor_SMD:R_0603_1608Metric_Pad0.98x0.95mm_HandSolder, B.Cu at (80.3, 156.2)
- added R405: 1k6, Resistor_SMD:R_0603_1608Metric_Pad0.98x0.95mm_HandSolder, B.Cu at (80.3, 157.9)
- added R406: 1k, Resistor_SMD:R_0603_1608Metric_Pad0.98x0.95mm_HandSolder, B.Cu at (88.9, 157.9)
- added R407: 1k, Resistor_SMD:R_0603_1608Metric_Pad0.98x0.95mm_HandSolder, B.Cu at (88.9, 156.2)
- added R408: 1k, Resistor_SMD:R_0603_1608Metric_Pad0.98x0.95mm_HandSolder, B.Cu at (133.1, 224.8)
- added R409: 1M, Resistor_SMD:R_0603_1608Metric_Pad0.98x0.95mm_HandSolder, B.Cu at (129.5, 224.8)
- added U401: YM2149, Package_DIP:DIP-40_W15.24mm_LongPads, F.Cu at (77.0, 151.2)
- added Y202: 4.433618MHz, Crystal:Crystal_HC49-4H_Vertical, F.Cu at (129.0, 215.9)
- added Y401: 2-4MHz, Crystal:Crystal_HC49-4H_Vertical, F.Cu at (129.0, 222.3)
- J101: value Screw_Terminal_01x02 -> Power +5V
- U102: footprint Package_SO:HTSSOP-20-1EP_4.4x6.5mm_P0.65mm_EP2.85x4mm -> Package_SO:SOP-20_7.5x12.8mm_P1.27mm; moved to B.Cu
- U202: footprint Package_SO:HTSSOP-14-1EP_4.4x5mm_P0.65mm_EP3.4x5mm_Mask3x3.1mm -> Package_SO:SOIC-14_3.9x8.7mm_P1.27mm; moved to B.Cu
- Y201: footprint Crystal:Crystal_HC52-6mm_Vertical -> Crystal:Crystal_HC49-4H_Vertical
- moved U301 71.1 mm to (142.9, 146.1), turned to 270 degrees
- moved U202 68.0 mm to (131.2, 229.6), turned to 270 degrees
- moved U302 60.8 mm to (142.9, 157.5), turned to 270 degrees
- moved U306 58.8 mm to (142.9, 203.2), turned to 270 degrees
- moved U303 53.4 mm to (142.9, 168.9), turned to 270 degrees
- moved U305 52.3 mm to (142.9, 191.8), turned to 270 degrees
- moved Y201 51.1 mm to (112.3, 146.9)
- moved U304 50.3 mm to (142.9, 180.3), turned to 270 degrees
- moved U102 49.8 mm to (108.0, 168.3), turned to 270 degrees
- moved U201 43.3 mm to (97.2, 151.1), turned to 0 degrees
- moved U203 36.9 mm to (107.4, 213.6), turned to 270 degrees
- moved U101 13.9 mm to (64.1, 151.1)
Connections:
- HDR101 pad 32: Net-(HDR101-Pad32) -> /~WR
- HDR101 pad 33: Net-(HDR101-Pad33) -> /~RD
- HDR102 pad 11: /~RD -> Net-(HDR102-Pad11)
- HDR102 pad 12: /~WR -> Net-(HDR102-Pad12)
- U101 pad 1: /~IOREQ -> /A1
- U101 pad 10: /A5 -> /~RD
- U101 pad 11: /A6 -> /~IOREQ
- U101 pad 14: /A7 -> /~M1
- U101 pad 15: Net-(U101-Pad15) -> /~VDP_RD
- U101 pad 16: Net-(U101-Pad16) -> /~VDP_WR
- U101 pad 17: Net-(U101-Pad17) -> /BDIR
- U101 pad 18: Net-(U101-Pad18) -> /BC1
- U101 pad 19: Net-(U101-Pad19) -> /IVL
- U101 pad 2: /~RD -> /A0
- U101 pad 21: /IVL -> Net-(U101-Pad21)
- U101 pad 22: /~VDP_WR -> Net-(U101-Pad22)
- U101 pad 23: /~VDP_RD -> Net-(U101-Pad23)
- U101 pad 3: /~WR -> /A3
- U101 pad 4: /~M1 -> /A2
- U101 pad 5: /A0 -> /A5
- U101 pad 6: /A1 -> /A4
- U101 pad 7: /A2 -> /A7
- U101 pad 8: /A3 -> /A6
- U101 pad 9: /A4 -> /~WR
- U102 pad 12: /D7 -> /D0
- U102 pad 13: /D6 -> /D1
- U102 pad 14: /D5 -> /D2
- U102 pad 15: /D4 -> /D3
- U102 pad 16: /D3 -> /D4
- U102 pad 17: /D2 -> /D5
- U102 pad 18: /D1 -> /D6
- U102 pad 19: /D0 -> /D7
- U102 pad 2: /D0 -> /D7
- U102 pad 3: /D1 -> /D6
- U102 pad 4: /D2 -> /D5
- U102 pad 5: /D3 -> /D4
- U102 pad 6: /D4 -> /D3
- U102 pad 7: /D5 -> /D2
- U102 pad 8: /D6 -> /D1
- U102 pad 9: /D7 -> /D0
- U202 pad 10: Net-(U202-Pad10) -> /SoundGen/CLK
- U202 pad 11: GND -> Net-(R408-Pad1)
- U202 pad 12: Net-(U202-Pad12) -> Net-(R408-Pad1)
- U202 pad 13: GND -> Net-(C404-Pad1)
Routing:
- net +5V: track 62.4 -> 369.1 mm, vias 0 -> 3
- net /A1: track 0.00 -> 102.6 mm, vias 0 -> 2
- net /A0: track 0.00 -> 101.0 mm, vias 0 -> 2
- net /D7: track 0.00 -> 99.8 mm, vias 0 -> 4
- net /D1: track 0.00 -> 91.2 mm, vias 0 -> 3
- net /D3: track 0.00 -> 89.8 mm, vias 0 -> 3
- net /D2: track 0.00 -> 87.4 mm, vias 0 -> 3
- net /D0: track 0.00 -> 87.1 mm, vias 0 -> 3
- net /D5: track 0.00 -> 85.2 mm, vias 0 -> 1
- net /D6: track 0.00 -> 83.9 mm, vias 0 -> 3
- net /D4: track 0.00 -> 80.8 mm, vias 0 -> 1
- net /SoundGen/CLK: track 0.00 -> 75.9 mm, vias 0 -> 1
- net /~RD: track 0.00 -> 74.9 mm, vias 0 -> 1
- net /~WR: track 0.00 -> 72.1 mm, vias 0 -> 1
- net /VDP/SYNCin: track 0.00 -> 67.1 mm, vias 0 -> 1
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- added copper zone on B.Cu, net GND
- added copper zone on F.Cu, net GND

Commit message: finishing
Parts:
- U201: value v9958 -> V9958
- moved U202 17.6 mm to (117.3, 218.7), turned to 0 degrees
- moved C225 8.69 mm to (119.1, 224.6), turned to 180 degrees
- moved C302 3.97 mm to (120.1, 156.6), turned to 90 degrees
- moved C214 1.54 mm to (101.1, 210.9), turned to 0 degrees
- moved C203 0.76 mm to (124.5, 216.7)
- moved C204 0.76 mm to (139.2, 216.7)
- moved C404 0.76 mm to (124.5, 223.0)
- moved C405 0.76 mm to (139.2, 223.0)
- moved R214 0.76 mm to (133.1, 219.2)
- moved R215 0.76 mm to (129.5, 219.2)
- moved R408 0.76 mm to (133.1, 225.6)
- moved R409 0.76 mm to (129.5, 225.6)
- moved Y202 0.76 mm to (129.0, 216.7)
- moved Y401 0.76 mm to (129.0, 223.0)
- moved R216 0.10 mm to (101.0, 161.7)
Routing:
- net +5V: track 369.1 -> 539.2 mm, vias 3 -> 4
- net /~M1: track 0.00 -> 99.6 mm, vias 0 -> 2
- net /~IOREQ: track 0.00 -> 95.2 mm, vias 0 -> 2
- net /~RST: track 0.00 -> 76.8 mm, vias 0 -> 1
- net /VDP/CAR-PAL: track 61.8 -> 11.2 mm, vias 2 -> 0
- net Net-(C402-Pad1): track 6.73 -> 56.9 mm, vias 2 -> 3
- net /~WAIT: track 0.00 -> 49.4 mm, vias 0 -> 1
- net Net-(C403-Pad1): track 6.73 -> 49.8 mm, vias 2 -> 3
- net /~INT: track 0.00 -> 40.5 mm, vias 0 -> 1
- net /SoundGen/CLK: track 75.9 -> 40.8 mm
- net /VDP/SYNCout: track 2.69 -> 29.7 mm, vias 0 -> 1
- net Net-(JP202-Pad2): track 0.00 -> 17.9 mm, vias 0 -> 2
- net GND: track 6.30 -> 14.0 mm, vias 12 -> 94
- net Net-(R408-Pad1): track 10.4 -> 17.9 mm
- net Net-(R214-Pad1): track 13.5 -> 20.9 mm
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Other:
- net class Medium added: clearance 0.127, trace_width 0.4, via_dia 0.889, via_drill 0.635
- board text added: "+5V"
- board text added: "0"
- board text added: "7"
- board text added: ">PAL"
- board text added: "CLK/2"
- board text added: "GND"
- board text added: "IM0"
- board text added: "IM1/2"
- board text added: "Marc Jacobi Canned Bytes 2021"
- board text added: "PortA"
- board text added: "PortB"
- board text added: "Video Audio"
- board text added: "Zalt Sound & Video v1.0"

Commit message: updates
Parts:
- removed JP101: Vector-Enable, Jumper:SolderJumper-3_P1.3mm_Open_RoundedPad1.0x1.5mm
- removed R101: 10k, Resistor_SMD:R_0603_1608Metric_Pad0.98x0.95mm_HandSolder
- added JP102: EnableIM, Connector_PinHeader_2.54mm:PinHeader_1x03_P2.54mm_Vertical, F.Cu at (54.1, 187.4)
- C217, C218, C219, C220, C221, C222: footprint Capacitor_SMD:CP_Elec_4x3 -> Capacitor_SMD:CP_Elec_6.3x7.7
- C402, C403: value 470uF -> 220uF; footprint Capacitor_SMD:CP_Elec_5x3 -> Capacitor_SMD:CP_Elec_6.3x7.7
- U102: footprint Package_SO:SOP-20_7.5x12.8mm_P1.27mm -> Package_SO:SOIC-20W_7.5x12.8mm_P1.27mm
- moved C403 15.7 mm to (51.7, 181.2)
- moved C220 8.15 mm to (66.4, 229.0), turned to 90 degrees
- moved C402 6.50 mm to (66.0, 188.6)
- moved C218 6.45 mm to (59.0, 228.9), turned to 90 degrees
- moved R230 4.96 mm to (71.0, 215.8), turned to 90 degrees
- moved C217 4.70 mm to (66.0, 196.2)
- moved R231 4.07 mm to (72.8, 219.2)
- moved C222 3.58 mm to (66.1, 219.2)
- moved R228 2.55 mm to (71.0, 208.3), turned to 90 degrees
- moved C219 2.42 mm to (66.1, 203.7)
- moved R229 2.31 mm to (72.5, 221.7)
- moved C221 1.48 mm to (66.1, 211.4)
- moved R227 1.31 mm to (71.6, 223.6)
- moved R226 0.64 mm to (71.0, 200.4), turned to 90 degrees
- moved R216 0.15 mm to (101.0, 161.5)
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Routing:
- net +5V: track 539.2 -> 519.1 mm, vias 4 -> 2
- net Net-(C403-Pad1): track 49.8 -> 67.0 mm
- net Net-(JP102-Pad2): track 4.95 -> 19.6 mm, vias 0 -> 1
- net Net-(C218-Pad1): track 3.77 -> 16.4 mm
- net /SoundGen/AudioR: track 8.24 -> 20.4 mm
- net Net-(C220-Pad1): track 2.86 -> 12.1 mm
- net /VDP/GREEN: track 6.73 -> 13.4 mm
- net /SoundGen/AudioL: track 5.67 -> 11.2 mm
- net Net-(R230-Pad1): track 36.7 -> 31.2 mm
- net Net-(R231-Pad1): track 37.8 -> 33.1 mm
- net /VDP/LUMA: track 6.68 -> 11.4 mm
- net Net-(R228-Pad1): track 28.9 -> 24.5 mm
- net Net-(JP101-Pad3): track 3.09 -> 0.00 mm
- net /VDP/BLUE: track 4.98 -> 7.68 mm
- net Net-(R229-Pad1): track 32.3 -> 29.8 mm
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Other:
- board text added: "<PAL"
- board text added: "IM0/2"
- board text added: "IM1"
- board text added: "PAL>"
- board text removed: ">PAL"
- board text removed: "IM0"
- board text removed: "IM1/2"
