File: Under Construction/VDP-Composite v0.1/Kicad/VDP-Composite.sch (KiCad schematic (older format))
At the start: 9 parts, among them J101 Screw_Terminal_01x02, U101 G22V10, U102 74HCT574

Commit message: progress
Parts:
- C101, C102: footprint Capacitor_SMD:C_1206_3216Metric_Pad1.33x1.80mm_HandSolder -> Capacitor_SMD:C_0603_1608Metric_Pad1.08x0.95mm_HandSolder
- J101: value Screw_Terminal_01x02 -> Power +5V
- R101: footprint Resistor_SMD:R_1206_3216Metric_Pad1.42x1.75mm_HandSolder -> Resistor_SMD:R_0603_1608Metric_Pad0.98x0.95mm_HandSolder
- U102: footprint Package_SO:HTSSOP-20-1EP_4.4x6.5mm_P0.65mm_EP2.85x4mm -> Package_SO:SOP-20_7.5x12.8mm_P1.27mm
Connections:
- net labels added: BC1, BDIR
- wire segments 93 -> 102
- no-connect marks 58 -> 56
Other:
- note removed: "Can use 16V8?"
- moved on the sheet: C101

Commit message: finishing
Other:
- note added: "Interrupt Vector Output Enable (IVOR) Activates when a Z80 CPU Interrupt \nAcknowledge Cycle is detected: ~M1~ and ~IOREQ~ both active."
- note removed: "Interrupt Vector Output Enable (IVOR) Activates when a Z80 CPU Interrupt \nAcknowledge Cycle is detected: ~M1~ and ~IOREQ~both active."
Changed lines of the file:
@@
 Interrupt Vecor Load (IVL)\nActivates when the correct IO Address is written to.
 Text Notes 950  6850 0    50   ~ 0
-Interrupt Vector Output Enable (IVOR) Activates when a Z80 CPU Interrupt \nAcknowledge Cycle is detected: ~M1~ and ~IOREQ~both active.
+Interrupt Vector Output Enable (IVOR) Activates when a Z80 CPU Interrupt \nAcknowledge Cycle is detected: ~M1~ and ~IOREQ~ both active.
 $Comp
 L Jumper:SolderJumper_3_Bridged12 JP101

Commit message: updates
Parts:
- removed JP101: Vector-Enable, Jumper:SolderJumper-3_P1.3mm_Open_RoundedPad1.0x1.5mm, symbol Jumper:SolderJumper_3_Bridged12
- removed R101: 10k, Resistor_SMD:R_0603_1608Metric_Pad0.98x0.95mm_HandSolder, symbol Device:R
- added JP102: EnableIM, Connector_PinHeader_2.54mm:PinHeader_1x03_P2.54mm_Vertical, symbol Jumper:Jumper_3_Bridged12
- U102: footprint Package_SO:SOP-20_7.5x12.8mm_P1.27mm -> Package_SO:SOIC-20W_7.5x12.8mm_P1.27mm
Changed lines of the file:
@@
 F 0 "U102" H 2700 6331 50  0000 C CNN
 F 1 "74HCT574" H 2700 6240 50  0000 C CNN
-F 2 "Package_SO:SOP-20_7.5x12.8mm_P1.27mm" H 2700 5350 50  0001 C CNN
+F 2 "Package_SO:SOIC-20W_7.5x12.8mm_P1.27mm" H 2700 5350 50  0001 C CNN
 F 3 "http://www.ti.com/lit/gpn/sn74HCT574" H 2700 5350 50  0001 C CNN
 	1    2700 5350
@@
 Text Notes 950  6850 0    50   ~ 0
 Interrupt Vector Output Enable (IVOR) Activates when a Z80 CPU Interrupt \nAcknowledge Cycle is detected: ~M1~ and ~IOREQ~ both active.
-$Comp
-L Jumper:SolderJumper_3_Bridged12 JP101
-U 1 1 60136017
-P 4350 6100
-F 0 "JP101" V 4396 6167 50  0000 L CNN
-F 1 "Vector-Enable" V 4305 6167 50  0000 L CNN
-F 2 "Jumper:SolderJumper-3_P1.3mm_Open_RoundedPad1.0x1.5mm" H 4350 6100 50  0001 C CNN
-F 3 "~" H 4350 6100 50  0001 C CNN
-	1    4350 6100
-	0    -1   -1   0
-$EndComp
 Wire Wire Line
 	4500 6100 4700 6100
@@
 L power:GND #PWR0114
 U 1 1 6013FC48
-P 4350 6300
-F 0 "#PWR0114" H 4350 6050 50  0001 C CNN
-F 1 "GND" H 4355 6127 50  0000 C CNN
-F 2 "" H 4350 6300 50  0001 C CNN
-F 3 "" H 4350 6300 50  0001 C CNN
-	1    4350 6300
-	1    0    0    -1
-$EndComp
-$Comp
-L Device:R R101
-U 1 1 601402BA
-P 4350 5750
-F 0 "R101" H 4420 5796 50  0000 L CNN
-F 1 "10k" H 4420 5705 50  0000 L CNN
-F 2 "Resistor_SMD:R_0603_1608Metric_Pad0.98x0.95mm_HandSolder" V 4280 5750 50  0001 C CNN
-F 3 "~" H 4350 5750 50  0001 C CNN
-	1    4350 5750
+P 4350 6350
+F 0 "#PWR0114" H 4350 6100 50  0001 C CNN
+F 1 "GND" H 4355 6177 50  0000 C CNN
+F 2 "" H 4350 6350 50  0001 C CNN
+F 3 "" H 4350 6350 50  0001 C CNN
+	1    4350 6350
 	1    0    0    -1
 $EndComp
@@
 L power:+5V #PWR0113
 U 1 1 601409A0
-P 4350 5600
-F 0 "#PWR0113" H 4350 5450 50  0001 C CNN
-F 1 "+5V" H 4365 5773 50  0000 C CNN
-F 2 "" H 4350 5600 50  0001 C CNN
-F 3 "" H 4350 5600 50  0001 C CNN
-	1    4350 5600
+P 4350 5850
+F 0 "#PWR0113" H 4350 5700 50  0001 C CNN
+F 1 "+5V" H 4365 6023 50  0000 C CNN
+F 2 "" H 4350 5850 50  0001 C CNN
+F 3 "" H 4350 5850 50  0001 C CNN
+	1    4350 5850
 	1    0    0    -1
 $EndComp
@@
 NoConn ~ 6500 4450
 NoConn ~ 6500 4350
+$Comp
+L Jumper:Jumper_3_Bridged12 JP102
+U 1 1 5FE574D4
+P 4350 6100
+F 0 "JP102" V 4396 6167 50  0000 L CNN
+F 1 "EnableIM" V 4305 6167 50  0000 L CNN
+F 2 "Connector_PinHeader_2.54mm:PinHeader_1x03_P2.54mm_Vertical" H 4350 6100 50  0001 C CNN
+F 3 "~" H 4350 6100 50  0001 C CNN
+	1    4350 6100
+	0    -1   -1   0
+$EndComp
 Wire Bus Line
 	1650 2650 1650 3750
