File: Under Construction/VDP-Composite v0.1/Kicad/VDP.sch (KiCad schematic (older format))
At the start: 76 parts, among them J201 SCART-F, J202 DIN-8, J203 Video (Yellow), J204 s-video, J205 AudioL (White), J206 AudioR (Red), U201 v9958, U202 74HCT04, U203 CXA1645, Y201 21.47727MHz, Y202 4.433618MHz

Commit message: progress
Parts:
- removed unit 5 of U202
- removed unit 6 of U202
- added J207: AVConn, Connector_IDC:IDC-Header_2x10_P2.54mm_Horizontal, symbol Connector_Generic:Conn_02x10_Counter_Clockwise
- C201, C204: footprint Capacitor_SMD:C_1206_3216Metric_Pad1.33x1.80mm_HandSolder -> Capacitor_THT:C_Disc_D6.0mm_W4.4mm_P5.00mm
- C202, C203, C205, C206, C207, C208, C210, C211, C212, C213, C214, C215, C216, C223, C224, C225, C226, C227: footprint Capacitor_SMD:C_1206_3216Metric_Pad1.33x1.80mm_HandSolder -> Capacitor_SMD:C_0603_1608Metric_Pad1.08x0.95mm_HandSolder
- C209: footprint Capacitor_SMD:CP_Elec_5x3 -> Capacitor_SMD:CP_Elec_4x3
- C217, C218, C219, C220, C221, C222: footprint Capacitor_SMD:C_1206_3216Metric_Pad1.33x1.80mm_HandSolder -> Capacitor_SMD:CP_Elec_4x3
- J203, J205, J206: footprint Connector_Coaxial:SMA_Molex_73251-1153_EdgeMount_Horizontal -> (none)
- R201, R202, R203, R204, R205, R206, R207, R208, R209, R210, R211, R212, R213, R214, R215, R216, R217, R218, R219, R220, R221, R222, R223, R224, R225, R226, R227, R228, R229, R230, R231, R232, R233, R234, R235, R236: footprint Resistor_SMD:R_1206_3216Metric_Pad1.42x1.75mm_HandSolder -> Resistor_SMD:R_0603_1608Metric_Pad0.98x0.95mm_HandSolder
- U202: footprint Package_SO:HTSSOP-14-1EP_4.4x5mm_P0.65mm_EP3.4x5mm_Mask3x3.1mm -> Package_SO:SOIC-14_3.9x8.7mm_P1.27mm
- U203: footprint fp -> Package_DIP:DIP-24_W10.16mm_LongPads
- Y201, Y202: footprint Crystal:Crystal_HC52-6mm_Vertical -> Crystal:Crystal_HC49-4H_Vertical
Connections:
- net labels added: AudioL, AudioR
- wire segments 395 -> 425
- no-connect marks 13 -> 11
Other:
- moved on the sheet: J201, J202, J203, J204, J205, J206, R232, R233, R234, R235

Commit message: updates
Parts:
- C217, C218, C219, C220, C221, C222: footprint Capacitor_SMD:CP_Elec_4x3 -> Capacitor_SMD:CP_Elec_6.3x7.7
- U201: value v9958 -> V9958
Changed lines of the file:
@@
 AR Path="/5FDC62A1/5FDC829A" Ref="U201"  Part="1"
 F 0 "U201" H 2500 5265 50  0000 C CNN
-F 1 "v9958" H 2500 5174 50  0000 C CNN
+F 1 "V9958" H 2500 5174 50  0000 C CNN
 F 2 "DIP178:DIP-64_1.78mm_W19.05mm" H 2150 5050 50  0001 C CNN
 F 3 "https://www.datasheets360.com/pdf/-6928505348629820723" H 1900 5400 50  0001 C CNN
@@
 F 0 "C218" H 8518 4746 50  0000 L CNN
 F 1 "220uF" H 8518 4655 50  0000 L CNN
-F 2 "Capacitor_SMD:CP_Elec_4x3" H 8438 4550 50  0001 C CNN
+F 2 "Capacitor_SMD:CP_Elec_6.3x7.7" H 8438 4550 50  0001 C CNN
 F 3 "~" H 8400 4700 50  0001 C CNN
 	1    8400 4700
@@
 F 0 "C220" H 8668 4896 50  0000 L CNN
 F 1 "220uF" H 8668 4805 50  0000 L CNN
-F 2 "Capacitor_SMD:CP_Elec_4x3" H 8588 4700 50  0001 C CNN
+F 2 "Capacitor_SMD:CP_Elec_6.3x7.7" H 8588 4700 50  0001 C CNN
 F 3 "~" H 8550 4850 50  0001 C CNN
 	1    8550 4850
@@
 F 0 "C222" H 8818 5046 50  0000 L CNN
 F 1 "220uF" H 8818 4955 50  0000 L CNN
-F 2 "Capacitor_SMD:CP_Elec_4x3" H 8738 4850 50  0001 C CNN
+F 2 "Capacitor_SMD:CP_Elec_6.3x7.7" H 8738 4850 50  0001 C CNN
 F 3 "~" H 8700 5000 50  0001 C CNN
 	1    8700 5000
@@
 F 0 "C217" H 8468 5346 50  0000 L CNN
 F 1 "220uF" H 8468 5255 50  0000 L CNN
-F 2 "Capacitor_SMD:CP_Elec_4x3" H 8388 5150 50  0001 C CNN
+F 2 "Capacitor_SMD:CP_Elec_6.3x7.7" H 8388 5150 50  0001 C CNN
 F 3 "~" H 8350 5300 50  0001 C CNN
 	1    8350 5300
@@
 F 0 "C219" H 8618 5496 50  0000 L CNN
 F 1 "220uF" H 8618 5405 50  0000 L CNN
-F 2 "Capacitor_SMD:CP_Elec_4x3" H 8538 5300 50  0001 C CNN
+F 2 "Capacitor_SMD:CP_Elec_6.3x7.7" H 8538 5300 50  0001 C CNN
 F 3 "~" H 8500 5450 50  0001 C CNN
 	1    8500 5450
@@
 F 0 "C221" H 8768 5646 50  0000 L CNN
 F 1 "220uF" H 8768 5555 50  0000 L CNN
-F 2 "Capacitor_SMD:CP_Elec_4x3" H 8688 5450 50  0001 C CNN
+F 2 "Capacitor_SMD:CP_Elec_6.3x7.7" H 8688 5450 50  0001 C CNN
 F 3 "~" H 8650 5600 50  0001 C CNN
 	1    8650 5600
