File: VDP Board v1.0 - locked/Kicad/VDP-Composite.kicad_pcb (KiCad board)
At the start: 2 copper layers, 99.7 x 99.7 mm, 113 parts, among them J101 Power +5V, J207 AVConn, J401 Ports, U101 G22V10, U102 74HCT574, U201 V9958, U202 74HCT04, U203 CXA1645, U301 D41464, U302 D41464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

Commit message: VDP in production
Other:
- board text added: "JLCJLCJLCJLC"
