File: VDP Board v1.0 - locked/Kicad/VDP-Composite.sch (KiCad schematic (older format))
At the start: 8 parts, among them J101 Power +5V, U101 G22V10, U102 74HCT574

Commit message: Ide prototype
Other:
- note added: "Interrupt Vector Output Enable (IVOE) Activates when a Z80 CPU Interrupt \nAcknowledge Cycle is detected: ~M1~ and ~IOREQ~ both active."
- note removed: "Interrupt Vector Output Enable (IVOR) Activates when a Z80 CPU Interrupt \nAcknowledge Cycle is detected: ~M1~ and ~IOREQ~ both active."
Changed lines of the file:
@@
 Interrupt Vecor Load (IVL)\nActivates when the correct IO Address is written to.
 Text Notes 950  6850 0    50   ~ 0
-Interrupt Vector Output Enable (IVOR) Activates when a Z80 CPU Interrupt \nAcknowledge Cycle is detected: ~M1~ and ~IOREQ~ both active.
+Interrupt Vector Output Enable (IVOE) Activates when a Z80 CPU Interrupt \nAcknowledge Cycle is detected: ~M1~ and ~IOREQ~ both active.
 Wire Wire Line
 	4500 6100 4700 6100
