File: Under Construction/IDE v0.1/Kicad/IDE.sch (KiCad schematic (older format))
At the start: 4 parts, among them J101 Power

Commit message: update
Other:
- note added: "Add\n- SD-card\n- PS2 keyboard / mouse (INT)\n- GamePort JoyStick (Dsub15)"
Changed lines of the file:
@@
 Text Label 5450 2700 0    50   ~ 0
 ~WAIT
+Text Notes 7050 6900 0    50   ~ 0
+Add\n- SD-card\n- PS2 keyboard / mouse (INT)\n- GamePort JoyStick (Dsub15)
 $EndSCHEMATC
