File: Under Construction/IDE v0.1/Kicad/IDE16 Interface.sch (KiCad schematic (older format))
At the start: 20 parts, among them J201 Conn_IDE40, Q201 BC547, Q202 BC547, U201 GAL16V8, U202 GAL16V8, U203 74HCT574, U204 74HC646, U205 74HC646

Commit message: cpm
Connections:
- net labels added: (LoByte), IODRY, IORDY, ~LoadVect, ~OutVect
- net labels removed: OutVEct, VectAddr
- wire segments 218 -> 219
- no-connect marks 5 -> 4
Changed lines of the file:
@@
 Wire Wire Line
 	9600 4250 9700 4250
-NoConn ~ 8000 3750
 $Comp
 L Device:R R203
@@
 ~WR
 Text Label 3750 4250 0    50   ~ 0
+~EnableHi
+Text Label 3750 4350 0    50   ~ 0
 ~EnableLo
-Text Label 3750 4350 0    50   ~ 0
-~EnableHi
 Text Label 3750 4450 0    50   ~ 0
 ~LatchLo
@@
 OutVect
 Text Label 3550 2400 0    50   ~ 0
-VectAddr
-Text Label 2250 4850 0    50   ~ 0
-VectAddr
-Text Label 3750 4850 0    50   ~ 0
-LoadVect
+~LoadVect
 Text Label 3750 4950 0    50   ~ 0
-OutVEct
+~OutVect
 Text Label 2250 4450 0    50   ~ 0
 ~M1
@@
 Text Label 3750 4750 0    50   ~ 0
 Interrupt
-NoConn ~ 3800 2500
 NoConn ~ 4050 4650
 Text Notes 7750 1650 0    50   ~ 0
@@
 Text Notes 3350 3150 0    50   ~ 0
 Wait to slow CPU \ndown to 8MHz?
-Wire Bus Line
-	1450 5450 1450 6200
-Wire Bus Line
-	1450 4100 1450 4850
 $Comp
 L 74HC646:74HC646 U205
@@
 	1    0    0    -1
 $EndComp
+Wire Wire Line
+	8000 3750 7600 3750
+Text Label 7650 3750 0    50   ~ 0
+IODRY
+Text Label 3550 2500 0    50   ~ 0
+IORDY
+Text Label 3750 4650 0    50   ~ 0
+(LoByte)
+NoConn ~ 3800 2200
+Wire Bus Line
+	1450 5450 1450 6200
+Wire Bus Line
+	1450 4100 1450 4850
+Text Label 2250 4850 0    50   ~ 0
+Sel
 $EndSCHEMATC

Commit message: Ide working prototype
Other:
- note added: "Cpu -> IDE command:\nLow-byte is passed through to IDE directly (8-bits only)"
- note removed: "Cpu -> IDE command:\nLow-byte is passed through to IDE directly (9-bits only)"
Changed lines of the file:
@@
 NoConn ~ 4050 4650
 Text Notes 7750 1650 0    50   ~ 0
-Cpu -> IDE command:\nLow-byte is passed through to IDE directly (9-bits only)
+Cpu -> IDE command:\nLow-byte is passed through to IDE directly (8-bits only)
 Text Notes 4050 7400 0    50   ~ 0
 Stores Interrupt Vector (IM2) or \nRST instruction (IM0) for IDE.
@@
 (LoByte)
 NoConn ~ 3800 2200
+Text Label 2250 4850 0    50   ~ 0
+Sel
 Wire Bus Line
 	1450 5450 1450 6200
 Wire Bus Line
 	1450 4100 1450 4850
-Text Label 2250 4850 0    50   ~ 0
-Sel
 $EndSCHEMATC

Commit message: Ide prototype
Parts:
- added R?: 10k, symbol Device:R
Connections:
- wire segments 219 -> 222
Other:
- note added: "Wait to slow CPU \ndown (IORDY)"
- note removed: "Wait to slow CPU \ndown to 8MHz?"
