File: CPU Board v1.0 - locked/Kicad/Z80 CPU Board.sch (KiCad schematic (older format))
At the start: 39 parts, among them IC101 UM61512A, IC102 UM61512A, IC103 UM61512A, IC104 UM61512A, IC105 Z80CPU, IC106 GLT725608, P101 CONN_02X10, P102 CONN_01X02, U101 74F573, U102 74F573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

Commit message: update (images)
Parts:
- C101, C102, C103, C104, C105, C106, C107, C108, C109: symbol C-RESCUE-Z80_CPU_Board -> Z80-CPU-Board-rescue:C-RESCUE-Z80_CPU_Board
- HDR101: symbol BUSHDR-A -> syshdr:BUSHDR-A
- HDR102: symbol BUSHDR-B -> syshdr:BUSHDR-B
- IC101, IC102, IC103, IC104: symbol UM61512A -> Z80-CPU-Board-rescue:UM61512A
- IC105: symbol Z80CPU -> Z80-CPU-Board-rescue:Z80CPU
- IC106: symbol GLT725608 -> G-Link-GLT725608:GLT725608
- P101: symbol CONN_02X10 -> Z80-CPU-Board-rescue:CONN_02X10
- P102: symbol CONN_01X02 -> Z80-CPU-Board-rescue:CONN_01X02
- R101, R102, R103, R104, R105, R106, R107, R108, R109, R110, R111, R112, R113, R114, R115, R116, R117: symbol R -> Device:R
- U101, U102: symbol 74F573 -> 74ls573:74F573
- U103: symbol 74HC245 -> My-74-Logic:74HC245

Commit message: atmega ide controller
Connections:
- net !RD: no longer HDR101.33 (RD), HDR102.11 (RD), IC101.24 (OE), IC102.24 (OE), IC103.24 (OE), IC104.24 (OE), IC105.21 (~RD~), R105.2
- net !BUSACK renamed ~BUSACK
- net !BUSREQ renamed ~BUSREQ
- net !CPU_CLK renamed ~CPU_CLK
- net !CPU_HALT renamed ~CPU_HALT
- net !CPU_INT renamed ~CPU_INT
- net !CPU_M1 renamed ~CPU_M1
- net !CPU_RESET renamed ~CPU_RESET
- net !CPU_WAIT renamed ~CPU_WAIT
- net !IOMapTableOE renamed ~IOMapTableOE
- net !IOREQ renamed ~IOREQ
- net !MBE0 renamed ~MBE0
- net !MBE1 renamed ~MBE1
- net !MBE2 renamed ~MBE2
- net !MBE3 renamed ~MBE3
- net !MEMREQ renamed ~MEMREQ
- net !MapTableData renamed ~MapTableData
- net !MapTableOE renamed ~MapTableOE
- net !MemMapEn renamed ~MemMapEn
- net !MemMapOE renamed ~MemMapOE
- net !MemMapWE renamed ~MemMapWE
- net !NMI renamed ~NMI
- net !REFRESH renamed ~REFRESH
- net !WR renamed ~WR
- new net ~RD: HDR101.33 (RD), HDR102.11 (RD), IC101.24 (OE), IC102.24 (OE), IC103.24 (OE), IC104.24 (OE), IC105.21 (~RD~), R105.2
Other:
- note added: "A->B = ~RD~"
- note added: "Address Translation (AT) \n~AT-IO~ => AT in IO mode (Active Low)\n~AT-IO~ = ~IOREQ~ & A[11..0] = $FFF\n\n~AT-IO-1~ => Set Memory Map Table\n~AT-IO-2~ => Set IO Map Table\n~AT-IO-3~ => Read/Write IO Table Data"
- note added: "Load = ~AT-IO-1~"
- note added: "Load = ~AT-IO-2~"
- note added: "Missed ~BUSREQ~ :-("
- note added: "R103-R106\nnot placed!"
- note added: "R110-R117\nnot placed!"
- note added: "~CE~ = ~AT-IO-3~"
- note added: "~MEM-RD~"
- note added: "~OE~ = !(~AT-IO-3~ & ~WR~) \n& !~RST~ (& 'boot release')"
- note added: "~OE~ = !~AT-IO-2~"
- note added: "~OE~ = ~AT-IO-2~"
- note added: "~WE~ = ~AT-IO-3~ & ~WR~"
- note removed: "/CE = /AT-IO-3"
- note removed: "/MEM-RD"
- note removed: "/OE = !(/AT-IO-3 & /WR) \n& !/RST (& 'boot release')"
- note removed: "/OE = !/AT-IO-2"
- note removed: "/OE = /AT-IO-2"
- note removed: "/WE = /AT-IO-3 & /WR"
- note removed: "A->B = /RD"
- note removed: "Address Translation (AT) \n/AT-IO => AT in IO mode (Active Low)\n/AT-IO = /IOREQ & A[11..0] = $FFF\n\n/AT-IO-1 => Set Memory Map Table\n/AT-IO-2 => Set IO Map Table\n/AT-IO-3 => Read/Write IO Table Data"
- note removed: "Load = /AT-IO-1"
- note removed: "Load = /AT-IO-2"
- note removed: "Missed !BUSREQ :-("
Changed lines of the file:
@@
 EESchema Schematic File Version 4
-LIBS:Z80 CPU Board-cache
-EELAYER 29 0
+EELAYER 30 0
 EELAYER END
 $Descr A3 16535 11693
@@
 	6900 4050 7000 3950
 Text Label 7000 1550 0    60   ~ 0
-!CPU_RESET
+~CPU_RESET
 Text Label 7000 1850 0    60   ~ 0
-!CPU_CLK
+~CPU_CLK
 Text Label 7000 2150 0    60   ~ 0
-!NMI
+~NMI
 Text Label 7000 2250 0    60   ~ 0
-!CPU_INT
+~CPU_INT
 Text Label 7000 2550 0    60   ~ 0
-!CPU_M1
+~CPU_M1
 Text Label 7000 2650 0    60   ~ 0
-!REFRESH
+~REFRESH
 Text Label 7000 2750 0    60   ~ 0
-!CPU_WAIT
+~CPU_WAIT
 Text Label 7000 2850 0    60   ~ 0
-!CPU_HALT
+~CPU_HALT
 Text Label 7000 3250 0    60   ~ 0
-!RD
+~RD
 Text Label 7000 3350 0    60   ~ 0
-!WR
+~WR
 Text Label 7000 3450 0    60   ~ 0
-!MEMREQ
+~MEMREQ
 Text Label 7000 3550 0    60   ~ 0
-!IOREQ
+~IOREQ
 Text Label 7000 3850 0    60   ~ 0
-!BUSREQ
+~BUSREQ
 Text Label 7000 3950 0    60   ~ 0
-!BUSACK
+~BUSACK
 $Comp
 L Z80-CPU-Board-rescue:UM61512A IC101
@@
 CPU_ME
 Text Label 3300 2150 2    60   ~ 0
-!MBE0
+~MBE0
 Text Label 3300 4200 2    60   ~ 0
-!MBE1
+~MBE1
 Text Label 6150 2150 2    60   ~ 0
-!MBE2
+~MBE2
 Text Label 6150 4200 2    60   ~ 0
-!MBE3
+~MBE3
 Entry Wire Line
 	3400 2750 3500 2650
@@
 	2650 4500 2750 4600
 Text Label 2650 2350 2    60   ~ 0
-!RD
+~RD
 Text Label 2650 2450 2    60   ~ 0
-!WR
+~WR
 Text Label 2650 4400 2    60   ~ 0
-!RD
+~RD
 Text Label 2650 4500 2    60   ~ 0
-!WR
+~WR
 Entry Wire Line
 	6800 2350 6900 2450
@@
 	6800 4500 6900 4600
 Text Label 6800 2350 2    60   ~ 0
-!RD
+~RD
 Text Label 6800 2450 2    60   ~ 0
-!WR
+~WR
 Text Label 6800 4400 2    60   ~ 0
-!RD
+~RD
 Text Label 6800 4500 2    60   ~ 0
-!WR
+~WR
 $Comp
 L Z80-CPU-Board-rescue:C-RESCUE-Z80_CPU_Board C101
@@
 	7300 7800 7400 7700
 Text Label 7250 7000 2    60   ~ 0
-!BUSACK
+~BUSACK
 Text Label 7250 7100 2    60   ~ 0
-!CPU_WAIT
+~CPU_WAIT
 Text Label 7250 7200 2    60   ~ 0
-!REFRESH
+~REFRESH
 Text Label 7250 7300 2    60   ~ 0
-!IOREQ
+~IOREQ
 Text Label 7250 7400 2    60   ~ 0
-!WR
+~WR
 Text Label 7250 7500 2    60   ~ 0
-!NMI
+~NMI
 Text Label 7250 7800 2    60   ~ 0
-!CPU_CLK
+~CPU_CLK
 Entry Wire Line
 	4750 6900 4850 7000
@@
 	4750 7700 4850 7800
 Text Label 4900 7000 0    60   ~ 0
-!BUSREQ
+~BUSREQ
 Text Label 4900 7100 0    60   ~ 0
-!CPU_HALT
+~CPU_HALT
 Text Label 4900 7200 0    60   ~ 0
-!CPU_M1
+~CPU_M1
 Text Label 4900 7300 0    60   ~ 0
-!MEMREQ
+~MEMREQ
 Text Label 4900 7400 0    60   ~ 0
-!RD
+~RD
 Text Label 4900 7500 0    60   ~ 0
-!CPU_INT
+~CPU_INT
 Text Label 4900 7800 0    60   ~ 0
-!CPU_RESET
+~CPU_RESET
 Entry Wire Line
 	3850 7050 3950 6950
@@
 	1850 8650 1950 8550
 Text Label 2000 8450 0    60   ~ 0
-!MEMREQ
+~MEMREQ
 Text Label 2000 8550 0    60   ~ 0
-!RD
+~RD
 Text Label 4100 8550 2    60   ~ 0
-!CPU_WAIT
+~CPU_WAIT
 Text Label 4050 8450 2    60   ~ 0
-!WR
+~WR
 $Comp
 L Z80-CPU-Board-rescue:GND-RESCUE-Z80_CPU_Board #PWR013
@@
 Addresses $0xxx - $Fxxx \nmapped to $00xxx - $FFxxx
 Text Notes 11450 2550 0    60   ~ 0
-Address Translation (AT) \n/AT-IO => AT in IO mode (Active Low)\n/AT-IO = /IOREQ & A[11..0] = $FFF\n\n/AT-IO-1 => Set Memory Map Table\n/AT-IO-2 => Set IO Map Table\n/AT-IO-3 => Read/Write IO Table Data
+Address Translation (AT) \n~AT-IO~ => AT in IO mode (Active Low)\n~AT-IO~ = ~IOREQ~ & A[11..0] = $FFF\n\n~AT-IO-1~ => Set Memory Map Table\n~AT-IO-2~ => Set IO Map Table\n~AT-IO-3~ => Read/Write IO Table Data
 Text Notes 14250 5450 2    60   ~ 0
-A->B = /RD
+A->B = ~RD~
 Text Notes 14250 5550 2    60   ~ 0
-/CE = /AT-IO-3
+~CE~ = ~AT-IO-3~
 Text Notes 13950 4250 0    60   ~ 0
-/OE = !(/AT-IO-3 & /WR) \n& !/RST (& 'boot release')
+~OE~ = !(~AT-IO-3~ & ~WR~) \n& !~RST~ (& 'boot release')
 Text Notes 13950 4350 0    60   ~ 0
-/WE = /AT-IO-3 & /WR
+~WE~ = ~AT-IO-3~ & ~WR~
 Entry Wire Line
 	15400 4500 15500 4600
@@
 D7
 Text Notes 12450 4400 0    60   ~ 0
-/MEM-RD
+~MEM-RD~
 $Comp
 L Z80-CPU-Board-rescue:C-RESCUE-Z80_CPU_Board C106
@@
 $EndComp
 Text Notes 11150 5900 0    60   ~ 0
-Load = /AT-IO-2
+Load = ~AT-IO-2~
 Text Notes 11150 6000 0    60   ~ 0
-/OE = /AT-IO-2
+~OE~ = ~AT-IO-2~
 Text Notes 14550 2450 0    60   ~ 0
 Boolean equations are on \na logic level (not physical)
 Text Notes 10200 4750 0    60   ~ 0
-Load = /AT-IO-1
+Load = ~AT-IO-1~
 Text Notes 10200 4850 0    60   ~ 0
-/OE = !/AT-IO-2
+~OE~ = !~AT-IO-2~
 NoConn ~ 5500 8500
 NoConn ~ 5500 8600
@@
 CPU_ME
 Text Label 13050 7450 0    60   ~ 0
-!MBE1
+~MBE1
 Text Label 13050 7550 0    60   ~ 0
-!MBE3
+~MBE3
 Text Label 11100 7450 0    60   ~ 0
-!MBE0
+~MBE0
 Text Label 11100 7550 0    60   ~ 0
-!MBE2
+~MBE2
 $Comp
 L Device:R R101
 U 1 1 56EF9C98
 P 8850 7450
-F 0 "R101" V 8930 7450 50  0000 C CNN
+F 0 "R101" V 8780 7450 50  0000 C CNN
 F 1 "10k" V 8850 7450 50  0000 C CNN
 F 2 "Resistors_SMD:R_0603_HandSoldering" V 8780 7450 50  0001 C CNN
@@
 U 1 1 56EF9D33
 P 8850 7600
-F 0 "R102" V 8930 7600 50  0000 C CNN
+F 0 "R102" V 8780 7600 50  0000 C CNN
 F 1 "10k" V 8850 7600 50  0000 C CNN
 F 2 "Resistors_SMD:R_0603_HandSoldering" V 8780 7600 50  0001 C CNN
@@
 	8200 8200 8700 8200
 Text Label 8250 7450 0    60   ~ 0
-!NMI
+~NMI
 Text Label 8250 7600 0    60   ~ 0
-!CPU_INT
+~CPU_INT
 Text Label 8250 7750 0    60   ~ 0
-!MEMREQ
+~MEMREQ
 Text Label 8250 7900 0    60   ~ 0
-!IOREQ
+~IOREQ
 Text Label 8250 8050 0    60   ~ 0
-!RD
+~RD
 Text Label 8250 8200 0    60   ~ 0
-!WR
+~WR
 $Comp
 L Device:R R107
@@
 	8200 8350 8700 8350
 Text Label 8250 8350 0    60   ~ 0
-!CPU_WAIT
+~CPU_WAIT
 Wire Wire Line
 	9000 7450 9100 7450
@@
 	11050 8150 11850 8150
 Text Label 11100 7650 0    60   ~ 0
-!MemMapWE
+~MemMapWE
 Text Label 11100 7750 0    60   ~ 0
-!MemMapEn
+~MemMapEn
 Text Label 11100 7850 0    60   ~ 0
 MapTableLd
@@
 SysCtrlTableSel
 Text Label 13050 7650 2    60   ~ 0
-!MemMapOE
+~MemMapOE
 Text Label 13050 7750 2    60   ~ 0
-!MapTableData
+~MapTableData
 Text Label 13050 7850 2    60   ~ 0
-!MapTableOE
+~MapTableOE
 Text Label 13050 7950 2    60   ~ 0
-!IOMapTableOE
+~IOMapTableOE
 Text Label 13050 8050 2    60   ~ 0
 SpareTableSel
@@
 MA18
 Text Notes 8150 7050 0    60   ~ 0
-Missed !BUSREQ :-(
+Missed ~BUSREQ~ :-(
 Wire Wire Line
 	7800 4500 7950 4500
@@
 Wire Wire Line
 	12050 4700 12050 4750
+Wire Notes Line
+	9000 7650 8700 7650
+Text Notes 9150 8150 0    60   ~ 0
+R103-R106\nnot placed!
+Text Notes 15400 2800 0    60   ~ 0
+R110-R117\nnot placed!
+Wire Notes Line
+	14050 2700 14050 3000
+Wire Notes Line
+	14050 3000 15350 3000
+Wire Notes Line
+	15350 3000 15350 2700
+Wire Notes Line
+	15350 2700 14050 2700
+Wire Notes Line
+	8710 7660 8710 8250
+Wire Notes Line
+	8710 8250 9000 8250
+Wire Notes Line
+	9000 8250 9000 7650
 Wire Wire Line
 	5350 2350 6800 2350
