File: Under Construction/IDE v0.2/Kicad/IDE_DMA.sch (KiCad schematic (older format))
At the start: 19 parts

Commit message: update
Parts:
- removed U?: 74HC245, symbol 74xx:74HC245
- removed U?: ATmega128A-AU, Package_QFP:TQFP-64_14x14mm_P0.8mm, symbol MCU_Microchip_ATmega:ATmega128A-AU
- removed U?: G22V10, symbol G22V10:G22V10
- added U?: ATmega2560-16AU, Package_QFP:TQFP-100_14x14mm_P0.5mm, symbol MCU_Microchip_ATmega:ATmega2560-16AU
- added U?: GAL16V8, symbol Logic_Programmable:GAL16V8
- U?: value 74ACT573 (fast) -> 74AHC573 (fast)
Connections:
- net labels added: IOEnable, IdeInt, IdeRdy, SDSel, ~BusSel, ~IdeRst, ~IdeSel0, ~IdeSel1
- net labels removed: ~BusEnable, ~IdeSel
- wire segments 204 -> 195
Other:
- note added: "(positive logic)\nOutIntVect = M1 & IOREQ\nRegWr = IOREQ & WR & A[4..7]\nRegRd = IOREQ & RD & A[4..7]\nWait = (RegRd | RegWr) & IOEnable"
- note added: "2N7000\nN-Channel MOSFET"
- note added: "Although the datasheet says to \nuse a fast AHC latch, I have it \nworking with a plain HCT type."
- note added: "IdeInt should go on an INT-pin"
- note added: "LED"
- note added: "OutIntVect handling checks if an \ninterrupt was issued then outputs \nthe vector or instruction. \nOtherwise it does nothing.\n"
- note added: "RTC \n- backup battery\n- what chip? DS1307?\n- what IO needed/protocol (I2C=TWI/SPI)\n- incl. SRAM (vbat)\n- for file time / general Z80 use"
- note added: "TODO:\nSD-Card\n- 3V3 regulator\n- (A)HC(T) buffers as level shifters\n- SPI port"
- note removed: "(positive logic)\nMEMRQ = BusEnable & (DMA_RD | DMA_WR) - .OE = BusEnable\nRD = BusEnable & DMA_RD - .OE = BusEnable\nWR = BusEnable & DMA_WR - .OE = BusEnable\nIdeEnable = !BusEnable\nDataDir = DMA_WR\nRegWr = IOREQ & WR & A[4..7]\nRegRd = IOREQ & RD & A[4..7]"
- note removed: "Shared between XRAM and IDE"
- moved on the sheet: C?, J?, JP?, U?, Y?
